File: crush-power-board.kicad_sch (KiCad schematic)
At the start: 8 parts

Commit message: added all power regulator circuits
Parts:
- added C? (x11): C, symbol Device:C
- added C?: C_Polarized_US, symbol Device:C_Polarized_US
- added L? (x2): L, symbol Device:L
- added R? (x9): R_US, symbol Device:R_US
Connections:
- net GND: now also U?.10 (PGND), U?.11 (PGND), U?.11 (PGND), U?.12 (SYNC), U?.14 (GND), U?.17 (PGND), U?.2 (ILIM), U?.30 (PGND), U?.4 (AGND), U?.9 (PGND), C?.2, C?.2, C?.2, C?.2, C?.2, C?.2, C?.2, C?.2, C?.2, R?.2, R?.2, R?.2, R?.2
- net +BATT: now reaches U?.1 (VCin)
- net +BATT: now also U?.13 (PVin), U?.15 (En), U?.16 (VDRV), U?.25 (Ilimit), U?.26 (VDD), U?.29 (VIN), U?.7 (VIN), U?.8 (VIN), U?.9 (VIN), C?.1, C?.1, C?.1, R?.2
- net at U?.12 (SW): now also U?.13 (SW), U?.14 (SW), L?.1
- net at U?.19 (SS): now also C?.1
- net PGOOD_SIC467: now reaches U?.2 (PGOOD)
- net at U?.20 (VOUT): now also C?.1, L?.2, R?.1
- net at U?.22 (VFB): now also R?.1, R?.2
- net at U?.23 (AGND): now also U?.28 (AGND)
- net at U?.24 (fsw): now also R?.1
- net at U?.27 (Mode): now also R?.1
- net at U?.4 (BOOT): now also C?.1
- net at U?.5 (PHASE): now also U?.6 (PHASE), C?.2
- net at U?.1 (FB): now also U?.8 (VSNS), C?.2, R?.1, R?.2
- net at U?.10 (VCC/LDO): now also C?.1, R?.1
- net at U?.12 (SW): now also C?.2, L?.1
- net at U?.14 (BOOT): now also C?.1
- net at U?.5 (TON/MODE): now also R?.1
- net PGood: now reaches U?.7 (Pgood)
- net PGood: now also R?.2
- net at U?.13 (BIAS): now also C?.1
- net at U?.15 (EN): now also R?.1
- net 3v3 at 600mA renamed 3V3_ 600MA
- new net 5Vo: C?.1, C?.1, C?.1, L?.2, R?.1
Other:
- moved on the sheet: C?, L?, R?, U?
