File: 3v3_reg.kicad_sch (KiCad schematic)
At the start: 13 parts, among them U4 BD9G341AEFJ

Commit message: Fixed a lot of components
Parts:
- C5, C6, C7, C8: footprint (none) -> Capacitor_SMD:C_0603_1608Metric
- L2: footprint (none) -> crush-power-footprints:IND_#B953AS-330M=P3
- R4, R5, R6, R7, R8, R9: footprint (none) -> Resistor_SMD:R_0201_0603Metric
Changed lines of the file:
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@@
       (effects (font (size 1.27 1.27)) (justify left))
     )
-    (property "Footprint" "" (at 150.8252 115.57 0)
+    (property "Footprint" "Capacitor_SMD:C_0603_1608Metric" (at 150.8252 115.57 0)
       (effects (font (size 1.27 1.27)) hide)
     )
@@
       (effects (font (size 1.27 1.27)))
     )
-    (property "Footprint" "" (at 147.32 79.0448 0)
+    (property "Footprint" "Capacitor_SMD:C_0603_1608Metric" (at 147.32 79.0448 0)
       (effects (font (size 1.27 1.27)) hide)
     )
@@
       (effects (font (size 1.27 1.27)) (justify left))
     )
-    (property "Footprint" "" (at 107.696 103.124 90)
+    (property "Footprint" "Resistor_SMD:R_0201_0603Metric" (at 107.696 103.124 90)
       (effects (font (size 1.27 1.27)) hide)
     )
@@
       (effects (font (size 1.27 1.27)) (justify left))
     )
-    (property "Footprint" "" (at 197.8152 104.14 0)
+    (property "Footprint" "Capacitor_SMD:C_0603_1608Metric" (at 197.8152 104.14 0)
       (effects (font (size 1.27 1.27)) hide)
     )
@@
       (effects (font (size 1.27 1.27)) (justify left))
     )
-    (property "Footprint" "" (at 93.6752 104.14 0)
+    (property "Footprint" "Capacitor_SMD:C_0603_1608Metric" (at 93.6752 104.14 0)
       (effects (font (size 1.27 1.27)) hide)
     )
@@
       (effects (font (size 1.27 1.27)) (justify left))
     )
-    (property "Footprint" "" (at 131.826 123.444 90)
+    (property "Footprint" "Resistor_SMD:R_0201_0603Metric" (at 131.826 123.444 90)
       (effects (font (size 1.27 1.27)) hide)
     )
@@
       (effects (font (size 1.27 1.27)) (justify left))
     )
-    (property "Footprint" "" (at 181.356 95.504 90)
+    (property "Footprint" "Resistor_SMD:R_0201_0603Metric" (at 181.356 95.504 90)
       (effects (font (size 1.27 1.27)) hide)
     )
@@
       (effects (font (size 1.27 1.27)))
     )
-    (property "Footprint" "" (at 161.29 88.9 0)
-      (effects (font (size 1.27 1.27)) hide)
-    )
-    (property "Datasheet" "~" (at 161.29 88.9 0)
+    (property "Footprint" "crush-power-footprints:IND_#B953AS-330M=P3" (at 161.29 88.9 0)
+      (effects (font (size 1.27 1.27)) hide)
+    )
+    (property "Datasheet" "https://www.digikey.com/en/products/detail/murata-electronics/B953AS-330M-P3/6205616" (at 161.29 88.9 0)
       (effects (font (size 1.27 1.27)) hide)
     )
@@
       (effects (font (size 1.27 1.27)) (justify left))
     )
-    (property "Footprint" "" (at 107.696 94.234 90)
+    (property "Footprint" "Resistor_SMD:R_0201_0603Metric" (at 107.696 94.234 90)
       (effects (font (size 1.27 1.27)) hide)
     )
@@
       (effects (font (size 1.27 1.27)) (justify left))
     )
-    (property "Footprint" "" (at 150.876 122.174 90)
+    (property "Footprint" "Resistor_SMD:R_0201_0603Metric" (at 150.876 122.174 90)
       (effects (font (size 1.27 1.27)) hide)
     )
@@
       (effects (font (size 1.27 1.27)) (justify left))
     )
-    (property "Footprint" "" (at 181.356 105.664 90)
-      (effects (font (size 1.27 1.27)) hide)
-    )
+    (property "Footprint" "Resistor_SMD:R_0201_0603Metric" (at 181.356 105.664 90)
+      (effects (font (size 1.27 1.27)) hide)
+    )

Commit message: Added extra footprints for diodes and capacitors
Parts:
- D1: footprint (none) -> crush-power-footprints:DIO_RR601BM4_ROM-L
Changed lines of the file:
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@@
       (effects (font (size 1.27 1.27)) (justify left))
     )
-    (property "Footprint" "" (at 147.32 92.71 0)
+    (property "Footprint" "crush-power-footprints:DIO_RR601BM4_ROM-L" (at 147.32 92.71 0)
       (effects (font (size 1.27 1.27)) hide)
     )
