File: 3v3_reg.kicad_sch (KiCad schematic)
At the start: 13 parts, among them U1 BD9G341AEFJ

Commit message: fixed some more footprints for resistors. 0201 -> 0603
Parts:
- R1, R2, R3, R4, R5, R6: footprint Resistor_SMD:R_0201_0603Metric -> Resistor_SMD:R_0603_1608Metric
Changed lines of the file:
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@@
       (effects (font (size 1.27 1.27)) (justify left))
     )
-    (property "Footprint" "Resistor_SMD:R_0201_0603Metric" (at 107.696 103.124 90)
+    (property "Footprint" "Resistor_SMD:R_0603_1608Metric" (at 107.696 103.124 90)
       (effects (font (size 1.27 1.27)) hide)
     )
@@
       (effects (font (size 1.27 1.27)) (justify left))
     )
-    (property "Footprint" "Resistor_SMD:R_0201_0603Metric" (at 131.826 123.444 90)
+    (property "Footprint" "Resistor_SMD:R_0603_1608Metric" (at 131.826 123.444 90)
       (effects (font (size 1.27 1.27)) hide)
     )
@@
       (effects (font (size 1.27 1.27)) (justify left))
     )
-    (property "Footprint" "Resistor_SMD:R_0201_0603Metric" (at 181.356 95.504 90)
+    (property "Footprint" "Resistor_SMD:R_0603_1608Metric" (at 181.356 95.504 90)
       (effects (font (size 1.27 1.27)) hide)
     )
@@
       (effects (font (size 1.27 1.27)) (justify left))
     )
-    (property "Footprint" "Resistor_SMD:R_0201_0603Metric" (at 107.696 94.234 90)
+    (property "Footprint" "Resistor_SMD:R_0603_1608Metric" (at 107.696 94.234 90)
       (effects (font (size 1.27 1.27)) hide)
     )
@@
       (effects (font (size 1.27 1.27)) (justify left))
     )
-    (property "Footprint" "Resistor_SMD:R_0201_0603Metric" (at 150.876 122.174 90)
+    (property "Footprint" "Resistor_SMD:R_0603_1608Metric" (at 150.876 122.174 90)
       (effects (font (size 1.27 1.27)) hide)
     )
@@
       (effects (font (size 1.27 1.27)) (justify left))
     )
-    (property "Footprint" "Resistor_SMD:R_0201_0603Metric" (at 181.356 105.664 90)
-      (effects (font (size 1.27 1.27)) hide)
-    )
+    (property "Footprint" "Resistor_SMD:R_0603_1608Metric" (at 181.356 105.664 90)
+      (effects (font (size 1.27 1.27)) hide)
+    )
